Commit message: переделала меши

File: spider_description/urdf/spider_macro.xacro (robot description, xacro)
@@ -118,5 +118,5 @@
         <!-- femur -->
         <joint name="joint_femur_${side}${position}" type="revolute">
-            <origin xyz="${coxa_length} 0.0 0.0" rpy="-${pi/2} 0 0.0"/>
+            <origin xyz="${coxa_length} 0.0 0.0" rpy="${pi/2} 0 0.0"/>
             <parent link="link_coxa_${side}${position}"/>
             <child link="link_femur_${side}${position}"/>
@@ -128,5 +128,5 @@
                 <origin xyz="0.0 0.0 0.0" rpy="0.0 0.0 0.0"/>
                 <geometry>
-                    <mesh filename="package://spider_description/meshes/femur_link.STL"/>
+                    <mesh filename="package://spider_description/meshes/2.STL"/>
                 </geometry>
                 <material name="">
@@ -137,5 +137,5 @@
                 <origin xyz="0.0 0.0 0.0" rpy="0.0 0.0 0.0" />
                 <geometry>
-                    <mesh filename="package://spider_description/meshes/femur_link.STL"/>
+                    <mesh filename="package://spider_description/meshes/2.STL"/>
                 </geometry>
                 <material name="">
@@ -160,5 +160,5 @@
         <!-- tibia -->
         <joint name="joint_tibia_${side}${position}" type="revolute">
-          <origin xyz="${femur_length} 0.0  0.0" rpy="${pi} 0.0 0.0"/>
+          <origin xyz="${femur_length} 0.0  0.0" rpy="0.0 0.0 0.0"/>
           <parent link="link_femur_${side}${position}"/>
           <child link="link_tibia_${side}${position}"/>
@@ -217,9 +217,9 @@
         </link>
     </xacro:macro>
-<xacro:leg side="r" position="r" x="-0.170" y="-0.110" angle="-${pi*3/4}" axis_femur="-1" axis_tibia="1" axis_coxa="1" mass="0.0207333939617734"/>
-<xacro:leg side="r" position="m" x="0.0" y="-0.1325" angle="-${pi/2}" axis_femur="-1" axis_tibia="1" axis_coxa="1" mass="0.0207333939617734"/>
-<xacro:leg side="r" position="f" x="0.170" y="-0.110" angle="-${pi/4}" axis_femur="-1" axis_tibia="1" axis_coxa="1" mass="0.04073339396177341"/>
-<xacro:leg side="l" position="r" x="-0.170" y="0.110" angle="${pi*3/4}" axis_femur="1" axis_tibia="-1" axis_coxa="1" mass="0.0207333939617734"/>
-<xacro:leg side="l" position="m" x="0.0" y="0.1325" angle="${pi/2}" axis_femur="1" axis_tibia="-1" axis_coxa="1" mass="0.0207333939617734"/>
-<xacro:leg side="l" position="f" x="0.170" y="0.110" angle="${pi/4}" axis_femur="1" axis_tibia="-1" axis_coxa="1" mass="0.04073339396177341"/>
+<xacro:leg side="r" position="r" x="-0.170" y="-0.110" angle="-${pi*3/4}" axis_femur="1" axis_tibia="1" axis_coxa="1" mass="0.0207333939617734"/>
+<xacro:leg side="r" position="m" x="0.0" y="-0.1325" angle="-${pi/2}" axis_femur="1" axis_tibia="1" axis_coxa="1" mass="0.0207333939617734"/>
+<xacro:leg side="r" position="f" x="0.170" y="-0.110" angle="-${pi/4}" axis_femur="1" axis_tibia="1" axis_coxa="1" mass="0.04073339396177341"/>
+<xacro:leg side="l" position="r" x="-0.170" y="0.110" angle="${pi*3/4}" axis_femur="1" axis_tibia="1" axis_coxa="1" mass="0.0207333939617734"/>
+<xacro:leg side="l" position="m" x="0.0" y="0.1325" angle="${pi/2}" axis_femur="1" axis_tibia="1" axis_coxa="1" mass="0.0207333939617734"/>
+<xacro:leg side="l" position="f" x="0.170" y="0.110" angle="${pi/4}" axis_femur="1" axis_tibia="1" axis_coxa="1" mass="0.04073339396177341"/>
 </robot>
