Commit message: газебо есть, но просто существует

File: spider_description/urdf/spider.ros2_control.xacro (robot description, xacro)
@@ -1,5 +1,5 @@
 <?xml version="1.0"?>
 <robot xmlns:xacro="http://www.ros.org/wiki/xacro">
-    <xacro:macro name="spider_ros2_control" params="name initial_positions_file">
+    <xacro:macro name="spider_ros2_control" params="name initial_positions_file ">
         <xacro:property name="initial_positions" value="${xacro.load_yaml(initial_positions_file)['initial_positions']}"/>
         <ros2_control name="${name}" type="system">

File: spider_description/urdf/spider.urdf.xacro (robot description, xacro)
@@ -2,5 +2,11 @@
 <robot name="spider" xmlns:xacro="http://ros.org/wiki/xacro">
   <xacro:arg name="initial_positions_file" default="initial_positions.yaml" />
-  <xacro:include filename="$(find spider_description)/urdf/spider_macro.xacro"/>
+  <xacro:arg name="path_meshes" default="file://$(find spider_description)/meshes" />
+  <xacro:arg name="format_meshes_stl" default="False" />
+  <xacro:include filename="$(find spider_description)/urdf/spider_macro.xacro" />
+  <xacro:spider_macro path_meshes="$(arg path_meshes)" format_meshes_stl="$(arg format_meshes_stl)"/>
+      <!-- <xacro:arg name="path_meshes" default="package://spider_description/meshes" />
+      <xacro:arg name="format_meshes_stl" default="True" />
+  </xacro:include> -->
   <xacro:include filename="$(find spider_description)/urdf/spider.ros2_control.xacro" />
   <xacro:spider_ros2_control name="SpiderHardwareInterface" initial_positions_file="$(arg initial_positions_file)"/>

File: spider_description/urdf/spider_macro.xacro (robot description, xacro)
@@ -1,4 +1,14 @@
 <?xml version="1.0" encoding="UTF-8" ?>
 <robot xmlns:xacro="http://ros.org/wiki/xacro" name="spider">
+<xacro:macro name="spider_macro" params="path_meshes format_meshes_stl">
+    <xacro:property name="format_meshes_stl_" value="${format_meshes_stl}"/>
+    <!-- <xacro:arg name="path_meshes"  default="package://spider_description/meshes"/>
+    <xacro:arg name="format_meshes_stl"  default="True"/> -->
+    <xacro:if value="${format_meshes_stl_}">
+        <xacro:property name="format" value=".STL"/>
+    </xacro:if>
+    <xacro:unless value="${format_meshes_stl_}">
+        <xacro:property name="format" value=".dae"/>
+    </xacro:unless>
     <!-- Link properties -->
     <!-- <xacro:property name="pi" value="3.1415926535897931"/> -->
@@ -26,5 +36,6 @@
             <origin xyz="0.0 0.0 0.0" rpy="0.0 0.0 0.0"/>
             <geometry>
-                <mesh filename="package://spider_description/meshes/base_link.STL" />
+                <!-- <mesh filename="package://spider_description/meshes/base_link.STL" /> -->
+                <mesh filename="${path_meshes}/base_link${format}" />
             </geometry>
             <material name="">
@@ -35,5 +46,6 @@
             <origin xyz="0.0 0.0 0.0" rpy="0.0 0.0 0.0"/>
             <geometry>
-                <mesh filename="package://spider_description/meshes/base_link.STL" />
+                <!-- <mesh filename="package://spider_description/meshes/base_link.STL" /> -->
+                <mesh filename="${path_meshes}/base_link${format}" />
             </geometry>
             <material name="">
@@ -86,5 +98,6 @@
                <origin xyz="0.0 0.0 0.0" rpy="0.0 0.0 0.0"/>
                <geometry>
-                   <mesh filename="package://spider_description/meshes/coxa_link.STL"/>
+                    <!-- <mesh filename="package://spider_description/meshes/coxa_link.STL"/> -->
+                    <mesh filename="${path_meshes}/coxa_link${format}" />
                </geometry>
                <material name="">
@@ -95,5 +108,6 @@
                <origin xyz="0.0 0.0 0.0" rpy="0.0 0.0 0.0" />
                <geometry>
-                   <mesh filename="package://spider_description/meshes/coxa_link.STL"/>
+                   <!-- <mesh filename="package://spider_description/meshes/coxa_link.STL"/> -->
+                   <mesh filename="${path_meshes}/coxa_link${format}" />
                </geometry>
                <material name="">
@@ -128,5 +142,6 @@
                 <origin xyz="0.0 0.0 0.0" rpy="0.0 0.0 0.0"/>
                 <geometry>
-                    <mesh filename="package://spider_description/meshes/2.STL"/>
+                    <!-- <mesh filename="package://spider_description/meshes/2.STL"/> -->
+                    <mesh filename="${path_meshes}/2${format}" />
                 </geometry>
                 <material name="">
@@ -137,5 +152,6 @@
                 <origin xyz="0.0 0.0 0.0" rpy="0.0 0.0 0.0" />
                 <geometry>
-                    <mesh filename="package://spider_description/meshes/2.STL"/>
+                    <!-- <mesh filename="package://spider_description/meshes/2.STL"/> -->
+                    <mesh filename="${path_meshes}/2${format}" />
                 </geometry>
                 <material name="">
@@ -170,5 +186,6 @@
                 <origin xyz="0.0 0.0 0.0" rpy="0.0 0.0 0.0"/>
                 <geometry>
-                    <mesh filename="package://spider_description/meshes/tibia_link.STL"/>
+                    <!-- <mesh filename="package://spider_description/meshes/tibia_link.STL"/> -->
+                    <mesh filename="${path_meshes}/tibia_link${format}" />
                 </geometry>
                 <material name="">
@@ -179,5 +196,6 @@
                 <origin xyz="0.0 0.0 0.0" rpy="0.0 0.0 0.0" />
                 <geometry>
-                    <mesh filename="package://spider_description/meshes/tibia_link.STL"/>
+                    <!-- <mesh filename="package://spider_description/meshes/tibia_link.STL"/> -->
+                    <mesh filename="${path_meshes}/tibia_link${format}" />
                 </geometry>
                 <material name="">
@@ -223,3 +241,4 @@
 <xacro:leg side="l" position="m" x="0.0" y="0.1325" angle="${pi/2}" axis_femur="1" axis_tibia="1" axis_coxa="1" mass="0.0207333939617734"/>
 <xacro:leg side="l" position="f" x="0.170" y="0.110" angle="${pi/4}" axis_femur="1" axis_tibia="1" axis_coxa="1" mass="0.04073339396177341"/>
+</xacro:macro>
 </robot>
